File: ch340G-usb-uart/ch340G-usb-uart.kicad_pcb (KiCad board)
At the start: 2 copper layers, 39.1 x 21.1 mm, 19 parts, among them J1 10118194-0001LF, J2 TTL OUT, U1 CH340G, Y1 12MHz

Commit message: added J2 Legends
Other:
- board text added: "+3V3"
- board text added: "+5V"
- board text added: "GND"
- board text added: "RXD"
- board text added: "TXD"
- board text added: "VCC_SEL"
Changed lines of the file:
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@@
   (gr_line (start 115.6 101) (end 115.6 79.9) (layer "Edge.Cuts") (width 0.1))
   (gr_line (start 154.7 101) (end 115.6 101) (layer "Edge.Cuts") (width 0.1))
+  (gr_text "VCC_SEL" (at 146.8 85.8) (layer "B.SilkS")
+    (effects (font (size 1 1) (thickness 0.15)) (justify mirror))
+  )
+  (gr_text "+5V" (at 148.6 83.3) (layer "B.SilkS")
+    (effects (font (size 1 1) (thickness 0.15)) (justify mirror))
+  )
+  (gr_text "+3V3" (at 148.2 88.3) (layer "B.SilkS")
+    (effects (font (size 1 1) (thickness 0.15)) (justify mirror))
+  )
+  (gr_text "GND" (at 148.3 96) (layer "B.SilkS")
+    (effects (font (size 1 1) (thickness 0.15)) (justify mirror))
+  )
+  (gr_text "TXD" (at 148.6 91) (layer "B.SilkS")
+    (effects (font (size 1 1) (thickness 0.15)) (justify mirror))
+  )
   (gr_text "CH340G USB TTL" (at 127.2 91) (layer "B.SilkS")
     (effects (font (size 1.5 1.5) (thickness 0.3)) (justify mirror))
   )
+  (gr_text "RXD" (at 148.4 93.4) (layer "B.SilkS")
+    (effects (font (size 1 1) (thickness 0.15)) (justify mirror))
+  )
   (gr_text "TX" (at 141.9 87.4) (layer "F.SilkS")
